File: CoCoDragonMultiPak.kicad_sch (KiCad schematic)
At the start: 57 parts, among them IC1 74LS245DWR, IC10 74LS74ADR, IC11 74LS153DR, IC12 74AHCT30D, IC13 GAL16V8, IC2 74LS367ADR, IC3 74LS367ADR, IC4 74LS367ADR, IC5 74LS367ADR, IC6 74LS367ADR, IC7 74LS374DWR, IC8 74LS368AD, IC9 74LS139ADR, J1 CARTRIDGE EDGE, J2 CARTRIDGE EDGE, J3 CARTRIDGE EDGE, J4 CARTRIDGE EDGE, J5 CARTRIDGE EDGE, J6 Barrel_Jack_MountingPin, SW1 DEFAULT SLOT, SW2 SW_DPDT_x2, U1 R-7812-0.5, U2 LM2596S-5

Commit message: switch gal for cpld
Parts:
- removed C15, C16, C17: 100nF, Capacitor_SMD:C_0805_2012Metric_Pad1.18x1.45mm_HandSolder, symbol Device:C_Small
- removed C2: 220uF, Capacitor_SMD:CP_Elec_6.3x5.4_Nichicon, symbol Device:C_Polarized_Small
- removed IC10: 74LS74ADR, Package_SO:SOIC-14_3.9x8.7mm_P1.27mm, symbol 74xx:74LS74
- removed IC12: 74AHCT30D, Package_SO:SOIC-14_3.9x8.7mm_P1.27mm, symbol 74xx:74LS30
- removed IC13: GAL16V8, Package_DIP:DIP-20_W7.62mm_LongPads, symbol Logic_Programmable:GAL16V8
- removed J1: CARTRIDGE EDGE, CoCoDragonMultiPak:EdgeConnector, symbol Connector_Generic:Conn_02x20_Counter_Clockwise
- removed J2: CARTRIDGE EDGE, CoCoDragonMultiPak:CardSocket, symbol Connector_Generic:Conn_02x20_Counter_Clockwise
- added C20: 220uF, Capacitor_SMD:CP_Elec_6.3x5.4_Nichicon, symbol Device:C_Polarized_Small
- added C21: 100nF, Capacitor_SMD:C_0805_2012Metric_Pad1.18x1.45mm_HandSolder, symbol Device:C_Small
- added D3: LED, LED_SMD:LED_0805_2012Metric_Pad1.15x1.40mm_HandSolder, symbol Device:LED
- added J1: Cartridge Edge, CoCoDragonMultiPak:EdgeConnector, symbol Connector_Generic:Conn_02x20_Odd_Even
- added J2: Cartridge Socket, CoCoDragonMultiPak:CardSocket, symbol Connector_Generic:Conn_02x20_Odd_Even
- added J7: JTAG, Connector_IDC:IDC-Header_2x05_P2.54mm_Vertical, symbol Connector_Generic:Conn_02x05_Odd_Even
- added R7: 4.7K, Resistor_SMD:R_0805_2012Metric_Pad1.20x1.40mm_HandSolder, symbol Device:R_Small
- added U3: ATF1504AS-xAx44, Package_QFP:TQFP-44_10x10mm_P0.8mm, symbol CPLD_Microchip:ATF1504AS-xAx44
- R1, R2, R3, R4: footprint Resistor_SMD:R_0805_2012Metric_Pad1.20x1.40mm_HandSolder -> Resistor_SMD:R_0603_1608Metric
Connections:
- net +12V: now also J2.1 (Pin_1), J2.2 (Pin_2)
- net +5V: now also C20.1, C21.1, J2.9 (Pin_9), U3.17 (VCC), U3.29 (VCC), U3.41 (VCC), U3.9 (VCC)
- net A0: now also J1.19 (Pin_19)
- net A1: now also J1.20 (Pin_20)
- net A10: now also J1.29 (Pin_29)
- net A11: now also J1.30 (Pin_30)
- net A12: now also J1.31 (Pin_31)
- net A13: now also J1.37 (Pin_37)
- net A14: now also J1.38 (Pin_38)
- net A15: now also J1.39 (Pin_39)
- net A2: now also J1.21 (Pin_21)
- net A3: now also J1.22 (Pin_22)
- net A4: now also J1.23 (Pin_23)
- net A5: now also J1.24 (Pin_24)
- net A6: now also J1.25 (Pin_25)
- net A7: now also J1.26 (Pin_26)
- net A8: now also J1.27 (Pin_27)
- net A9: now also J1.28 (Pin_28)
- net CTRL1: now also U3.2 (I/O)
- net D0: now also J1.10 (Pin_10)
- net D1: now also J1.11 (Pin_11)
- net D2: now also J1.12 (Pin_12)
- net D3: now also J1.13 (Pin_13)
- net D4: now also J1.14 (Pin_14)
- net D5: now also J1.15 (Pin_15)
- net D6: now also J1.16 (Pin_16)
- net D7: now also J1.17 (Pin_17)
- net E: now also J1.6 (Pin_6)
- net ENREG: now also U3.18 (I/O)
- net ENSW: now also U3.8 (I/O)
- net EXTSND: now also J1.35 (Pin_35), J2.35 (Pin_35)
- net GND: now also C20.2, C21.2, D3.1 (K), J1.33 (Pin_33), J1.34 (Pin_34), J2.33 (Pin_33), J2.34 (Pin_34), J7.10 (Pin_10), J7.2 (Pin_2), J7.4 (Pin_4), J7.6 (Pin_6), J7.8 (Pin_8), U3.16 (GND), U3.24 (GND), U3.36 (GND), U3.4 (GND)
- net IA0: now also J2.19 (Pin_19), U3.35 (I/O/GCLK3)
- net IA1: now also J2.20 (Pin_20), U3.42 (I/O)
- net IA10: now also J2.29 (Pin_29), U3.28 (I/O)
- net IA11: now also J2.30 (Pin_30), U3.39 (I/GCLR)
- net IA12: now also J2.31 (Pin_31), U3.15 (I/O)
- net IA13: now also J2.37 (Pin_37), U3.19 (I/O/PD2)
- net IA14: now also J2.38 (Pin_38), U3.25 (I/O)
- net IA15: now also J2.39 (Pin_39), U3.33 (I/O)
- net IA2: now also J2.21 (Pin_21), U3.34 (I/O)
- net IA3: now also J2.22 (Pin_22), U3.43 (I/O)
- net IA4: now also J2.23 (Pin_23), U3.10 (I/O)
- net IA5: now also J2.24 (Pin_24), U3.11 (I/O)
- net IA6: now also J2.25 (Pin_25), U3.12 (I/O)
- net IA7: now also J2.26 (Pin_26), U3.31 (I/O)
- net IA8: now also J2.27 (Pin_27), U3.20 (I/O)
- net IA9: now also J2.28 (Pin_28), U3.14 (I/O)
- net ID0: now also J2.10 (Pin_10)
- net ID1: now also J2.11 (Pin_11)
- net ID2: now also J2.12 (Pin_12)
- net ID3: now also J2.13 (Pin_13)
- net ID4: now also J2.14 (Pin_14)
- net ID5: now also J2.15 (Pin_15)
- net ID6: now also J2.16 (Pin_16)
- net ID7: now also J2.17 (Pin_17)
- net IE: now also J2.6 (Pin_6), U3.23 (I/O)
- net IQ: now also J2.7 (Pin_7), U3.22 (I/O)
- net IR/~{W}: now also J2.18 (Pin_18), U3.21 (I/O)
- net I~{CTS}: now also U3.13 (I/O)
- net I~{RESET}: now also J2.5 (Pin_5), J7.1 (Pin_1), U3.30 (I/O)
- net LOADREG: now also U3.37 (I/GCLK1)
- net Q: now also J1.7 (Pin_7)
- net R/~{W}: now also J1.18 (Pin_18)
- net ~{CART1}: now also J2.8 (Pin_8)
- net ~{CART}: now also J1.8 (Pin_8)
- net ~{CTS1}: now also J2.32 (Pin_32)
- net ~{CTS}: now also J1.32 (Pin_32)
- net ~{ENBUS}: now also U3.5 (I/O/PD1)
- net ~{ENREAD}: now also U3.3 (I/O)
- net ~{HALT}: now also J1.3 (Pin_3), J2.3 (Pin_3)
- net ~{NMI}: now also J1.4 (Pin_4), J2.4 (Pin_4)
- net ~{P21}: now also J2.36 (Pin_36)
- net ~{P2}: now also J1.36 (Pin_36)
- net ~{RESET}: now also J1.5 (Pin_5)
- net ~{SLEN}: now also J1.40 (Pin_40), J2.40 (Pin_40), U3.40 (I/OE2/GCLK2)
- new net: D3.2 (A), R7.2
- new net +5VA: J1.9 (Pin_9), R7.1
- new net TCK: J7.9 (Pin_9), U3.26 (I/O/TCK)
- new net TDI: J7.3 (Pin_3), U3.1 (I/O/TDI)
- new net TDO: J7.5 (Pin_5), U3.32 (I/O/TDO)
- new net TMS: J7.7 (Pin_7), U3.7 (I/O/TMS)
- no-connect marks 13 -> 14
Other:
- note removed: "X"
- moved on the sheet: C10, C11, C13, C14, C18, C19, C5, C6, C7, C8, C9, D4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
