File: CoCoDragonMultiPak.kicad_sch (KiCad schematic)
At the start: 57 parts, among them IC1 74LS245DWR, IC10 74LS74ADR, IC11 74LS153DR, IC12 74AHCT30D, IC13 GAL16V8, IC2 74LS367ADR, IC3 74LS367ADR, IC4 74LS367ADR, IC5 74LS367ADR, IC6 74LS367ADR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

Commit message: revise for production
Connections:
- net CTRL1 renamed ~{ENWRITE}
