File: CoCoDragonMultiPak.kicad_pcb (KiCad board)
At the start: 2 copper layers, 137.7 x 171.2 mm, 58 parts, among them IC1 74LS245DWR, IC10 74LS74ADR, IC11 74LS153DR, IC12 74AHCT30D, IC13 GAL16V8, IC2 74LS367ADR, IC3 74LS367ADR, IC4 74LS367ADR, IC5 74LS367ADR, IC6 74LS367ADR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

Commit message: revise for production
Parts:
- moved C18 28.7 mm to (100.5, 62.5), turned to 90 degrees
- moved C2 15.1 mm to (91.3, 120.8), turned to 180 degrees
Connections:
- net /CTRL1 renamed /~{ENWRITE}
Routing:
- net /RECTIFIED_POWER: track 62.7 -> 48.0 mm
- net /REGS1: track 134.2 -> 126.6 mm, vias 6 -> 4
- net Net-(SW2B-B): track 22.9 -> 18.0 mm
- net /~{ENWRITE}: track 126.4 -> 131.1 mm, vias 4 -> 3
- net /I~{CTS}: track 55.6 -> 52.8 mm, vias 4 -> 2
- net +5V: track 684.6 -> 686.7 mm
- net /~{CTS4}: track 89.4 -> 87.7 mm
- net /AC2: track 24.2 -> 25.8 mm
- net /AC1: track 28.7 -> 29.8 mm
- net /ENSW: track 17.6 -> 16.7 mm
- net /~{RESET}: track 200.1 -> 201.0 mm
- net /IR/~{W}: track 226.1 -> 225.2 mm
- net /~{P24}: track 102.9 -> 102.2 mm
- net /~{CART3}: track 66.3 -> 65.6 mm
- net /~{CART}: track 125.7 -> 126.3 mm
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Other:
- board size 137.7 x 171.2 mm -> 138 x 171.2 mm
- board text added: "Version 1.0"
- board text removed: "Version 0.1"
